Commit message: 1.修正URDF命名错误 2.添加LICENSE

File: apex_hand_left/apex_hand_left.urdf (robot description, URDF)
Before this commit: robot Apex_hand_left, 47 links, 46 joints
Links:
- removed link Palm_link_left
- removed link f0_link0
- removed link f0_link1
- removed link f0_link2
- removed link f0_link2sensor
- removed link f0_link3
- removed link f0_link3sensor
- removed link f0_link4
- removed link f0_link4sensor
- removed link f0_pad
- removed link f0_tip
- removed link f1_link0
- removed link f1_link1
- removed link f1_link1sensor
- removed link f1_link2
- removed link f1_link2sensor
- removed link f1_link3
- removed link f1_link3sensor
- removed link f1_pad
- removed link f1_tip
- removed link f2_link0
- removed link f2_link1
- removed link f2_link1sensor
- removed link f2_link2
- removed link f2_link2sensor
- removed link f2_link3
- removed link f2_link3sensor
- removed link f2_pad
- removed link f2_tip
- removed link f3_link0
- removed link f3_link1
- removed link f3_link1sensor
- removed link f3_link2
- removed link f3_link2sensor
- removed link f3_link3
- removed link f3_link3sensor
- removed link f3_pad
- removed link f3_tip
- removed link f4_link0
- removed link f4_link1
- removed link f4_link1sensor
- removed link f4_link2
- removed link f4_link2sensor
- removed link f4_link3
- removed link f4_link3sensor
- removed link f4_pad
- removed link f4_tip
- added link left_index_link_0, mass 0.0187941572496829; collision mesh filename=./meshes/left_index_link_0.STL; visual mesh filename=./meshes/left_index_link_0.STL
- added link left_index_link_1, mass 0.0290954766878052; collision mesh filename=./meshes/left_index_link_1.STL; visual mesh filename=./meshes/left_index_link_1.STL
- added link left_index_link_2, mass 0.0111427111396244; collision mesh filename=./meshes/left_index_link_2.STL; visual mesh filename=./meshes/left_index_link_2.STL
- added link left_index_link_3, mass 0.00523283787432778; collision mesh filename=./meshes/left_index_link_3.STL; visual mesh filename=./meshes/left_index_link_3.STL
- added link left_index_pad, mass 8.20481262582146E-06; collision mesh filename=./meshes/left_index_pad.STL; visual mesh filename=./meshes/left_index_pad.STL
- added link left_index_tactile_0, mass 0.00892665816513553; collision mesh filename=./meshes/left_index_tactile_0.STL; visual mesh filename=./meshes/left_index_tactile_0.STL
- added link left_index_tactile_1, mass 0.00363566683984855; collision mesh filename=./meshes/left_index_tactile_1.STL; visual mesh filename=./meshes/left_index_tactile_1.STL
- added link left_index_tactile_2, mass 0.00986650295375492; collision mesh filename=./meshes/left_index_tactile_2.STL; visual mesh filename=./meshes/left_index_tactile_2.STL
- added link left_index_tip, mass 8.20481262582146E-06; collision mesh filename=./meshes/left_index_tip.STL; visual mesh filename=./meshes/left_index_tip.STL
- added link left_middle_link_0, mass 0.0187941572496829; collision mesh filename=./meshes/left_middle_link_0.STL; visual mesh filename=./meshes/left_middle_link_0.STL
- added link left_middle_link_1, mass 0.0290954766872579; collision mesh filename=./meshes/left_middle_link_1.STL; visual mesh filename=./meshes/left_middle_link_1.STL
- added link left_middle_link_2, mass 0.0111427111396244; collision mesh filename=./meshes/left_middle_link_2.STL; visual mesh filename=./meshes/left_middle_link_2.STL
- added link left_middle_link_3, mass 0.00520913037318323; collision mesh filename=./meshes/left_middle_link_3.STL; visual mesh filename=./meshes/left_middle_link_3.STL
- added link left_middle_pad, mass 8.20481262582145E-06; collision mesh filename=./meshes/left_middle_pad.STL; visual mesh filename=./meshes/left_middle_pad.STL
- added link left_middle_tactile_0, mass 0.00892665695013671; collision mesh filename=./meshes/left_middle_tactile_0.STL; visual mesh filename=./meshes/left_middle_tactile_0.STL
- added link left_middle_tactile_1, mass 0.00363566690746592; collision mesh filename=./meshes/left_middle_tactile_1.STL; visual mesh filename=./meshes/left_middle_tactile_1.STL
- added link left_middle_tactile_2, mass 0.00986650294179115; collision mesh filename=./meshes/left_middle_tactile_2.STL; visual mesh filename=./meshes/left_middle_tactile_2.STL
- added link left_middle_tip, mass 8.20481262582144E-06; collision mesh filename=./meshes/left_middle_tip.STL; visual mesh filename=./meshes/left_middle_tip.STL
- added link left_palm_link, mass 0.262853650060054; collision mesh filename=./meshes/left_palm_link.STL; visual mesh filename=./meshes/left_palm_link.STL
- added link left_pinky_link_0, mass 0.0187941572496829; collision mesh filename=./meshes/left_pinky_link_0.STL; visual mesh filename=./meshes/left_pinky_link_0.STL
- added link left_pinky_link_1, mass 0.0290954766878052; collision mesh filename=./meshes/left_pinky_link_1.STL; visual mesh filename=./meshes/left_pinky_link_1.STL
- added link left_pinky_link_2, mass 0.0111427111396244; collision mesh filename=./meshes/left_pinky_link_2.STL; visual mesh filename=./meshes/left_pinky_link_2.STL
- added link left_pinky_link_3, mass 0.00518541203449777; collision mesh filename=./meshes/left_pinky_link_3.STL; visual mesh filename=./meshes/left_pinky_link_3.STL
- added link left_pinky_pad, mass 8.20481262582147E-06; collision mesh filename=./meshes/left_pinky_pad.STL; visual mesh filename=./meshes/left_pinky_pad.STL
- added link left_pinky_tactile_0, mass 0.00892665816512027; collision mesh filename=./meshes/left_pinky_tactile_0.STL; visual mesh filename=./meshes/left_pinky_tactile_0.STL
- added link left_pinky_tactile_1, mass 0.00363566688943969; collision mesh filename=./meshes/left_pinky_tactile_1.STL; visual mesh filename=./meshes/left_pinky_tactile_1.STL
- added link left_pinky_tactile_2, mass 0.00986650302255517; collision mesh filename=./meshes/left_pinky_tactile_2.STL; visual mesh filename=./meshes/left_pinky_tactile_2.STL
- added link left_pinky_tip, mass 8.20481262582144E-06; collision mesh filename=./meshes/left_pinky_tip.STL; visual mesh filename=./meshes/left_pinky_tip.STL
- added link left_ring_link_0, mass 0.0187941572496829; collision mesh filename=./meshes/left_ring_link_0.STL; visual mesh filename=./meshes/left_ring_link_0.STL
- added link left_ring_link_1, mass 0.0290954766872579; collision mesh filename=./meshes/left_ring_link_1.STL; visual mesh filename=./meshes/left_ring_link_1.STL
- added link left_ring_link_2, mass 0.0111427111396243; collision mesh filename=./meshes/left_ring_link_2.STL; visual mesh filename=./meshes/left_ring_link_2.STL
- added link left_ring_link_3, mass 0.00518541203449776; collision mesh filename=./meshes/left_ring_link_3.STL; visual mesh filename=./meshes/left_ring_link_3.STL
- added link left_ring_pad, mass 8.20481262582145E-06; collision mesh filename=./meshes/left_ring_pad.STL; visual mesh filename=./meshes/left_ring_pad.STL
- added link left_ring_tactile_0, mass 0.00892665816509035; collision mesh filename=./meshes/left_ring_tactile_0.STL; visual mesh filename=./meshes/left_ring_tactile_0.STL
- added link left_ring_tactile_1, mass 0.0036356669074622; collision mesh filename=./meshes/left_ring_tactile_1.STL; visual mesh filename=./meshes/left_ring_tactile_1.STL
- added link left_ring_tactile_2, mass 0.00986650313583958; collision mesh filename=./meshes/left_ring_tactile_2.STL; visual mesh filename=./meshes/left_ring_tactile_2.STL
- added link left_ring_tip, mass 8.20481262582146E-06; collision mesh filename=./meshes/left_ring_tip.STL; visual mesh filename=./meshes/left_ring_tip.STL
- added link left_thumb_link_0, mass 0.0109675846438251; collision mesh filename=./meshes/left_thumb_link_0.STL; visual mesh filename=./meshes/left_thumb_link_0.STL
- added link left_thumb_link_1, mass 0.0155120351654751; collision mesh filename=./meshes/left_thumb_link_1.STL; visual mesh filename=./meshes/left_thumb_link_1.STL
- added link left_thumb_link_2, mass 0.0324231796920109; collision mesh filename=./meshes/left_thumb_link_2.STL; visual mesh filename=./meshes/left_thumb_link_2.STL
- added link left_thumb_link_3, mass 0.0183837211151652; collision mesh filename=./meshes/left_thumb_link_3.STL; visual mesh filename=./meshes/left_thumb_link_3.STL
- added link left_thumb_link_4, mass 0.00765584782571519; collision mesh filename=./meshes/left_thumb_link_4.STL; visual mesh filename=./meshes/left_thumb_link_4.STL
- added link left_thumb_pad, mass 8.20481262582145E-06; collision mesh filename=./meshes/left_thumb_pad.STL; visual mesh filename=./meshes/left_thumb_pad.STL
- added link left_thumb_tactile_0, mass 0.0359955765510153; collision mesh filename=./meshes/left_thumb_tactile_0.STL; visual mesh filename=./meshes/left_thumb_tactile_0.STL
- added link left_thumb_tactile_1, mass 0.00938453556455443; collision mesh filename=./meshes/left_thumb_tactile_1.STL; visual mesh filename=./meshes/left_thumb_tactile_1.STL
- added link left_thumb_tactile_2, mass 0.00986648442614148; collision mesh filename=./meshes/left_thumb_tactile_2.STL; visual mesh filename=./meshes/left_thumb_tactile_2.STL
- added link left_thumb_tip, mass 8.20481262582146E-06; collision mesh filename=./meshes/left_thumb_tip.STL; visual mesh filename=./meshes/left_thumb_tip.STL
Joints:
- removed joint f0_joint0
- removed joint f0_joint1
- removed joint f0_joint2
- removed joint f0_joint2sensor
- removed joint f0_joint3
- removed joint f0_joint3sensor
- removed joint f0_joint4
- removed joint f0_joint4sensor
- removed joint f0_pad
- removed joint f0_tip
- removed joint f1_joint0
- removed joint f1_joint1
- removed joint f1_joint1sensor
- removed joint f1_joint2
- removed joint f1_joint2sensor
- removed joint f1_joint3
- removed joint f1_joint3sensor
- removed joint f1_pad
- removed joint f1_tip
- removed joint f2_joint0
- removed joint f2_joint1
- removed joint f2_joint2
- removed joint f2_joint2sensor
- removed joint f2_joint3
- removed joint f2_joint3sensor
- removed joint f2_jont1sensor
- removed joint f2_pad
- removed joint f2_tip
- removed joint f3_joint0
- removed joint f3_joint1
- removed joint f3_joint1sensor
- removed joint f3_joint2
- removed joint f3_joint2sensor
- removed joint f3_joint3
- removed joint f3_joint3sensor
- removed joint f3_pad
- removed joint f3_tip
- removed joint f4_joint0
- removed joint f4_joint1
- removed joint f4_joint1sensor
- removed joint f4_joint2
- removed joint f4_joint2sensor
- removed joint f4_joint3
- removed joint f4_joint3sensor
- removed joint f4_pad
- removed joint f4_tip
- added joint left_index_j0: type revolute, parent left_palm_link, child left_index_link_0, origin xyz=0.0069979 -0.034496 0.1155 rpy=3.1416 -1.5708 0, axis 0 0 1, limit lower=-0.436 upper=0.436 effort=0 velocity=8.7266
- added joint left_index_j1: type revolute, parent left_index_link_0, child left_index_link_1, origin xyz=0.016 0 0 rpy=1.5708 0 0, axis 0 0 1, limit lower=-0.349 upper=1.5708 effort=0 velocity=8.7266
- added joint left_index_j1_sensor: type fixed, parent left_index_link_1, child left_index_tactile_0, origin xyz=0 0 0 rpy=0 0 0, axis 0 0 0
- added joint left_index_j2: type revolute, parent left_index_link_1, child left_index_link_2, origin xyz=0.045 0 0 rpy=0 0 0, axis 0 0 1, limit lower=-0.0873 upper=1.745 effort=0 velocity=8.7266
- added joint left_index_j2_sensor: type fixed, parent left_index_link_2, child left_index_tactile_1, origin xyz=0 0 0 rpy=0 0 0, axis 0 0 0
- added joint left_index_j3: type revolute, parent left_index_link_2, child left_index_link_3, origin xyz=0.025 0 0 rpy=0 0 0, axis 0 0 1, limit lower=-0.0873 upper=1.745 effort=0 velocity=8.7266, mimic joint=left_index_j2 multiplier=1.0 offset=0
- added joint left_index_j3_sensor: type fixed, parent left_index_link_3, child left_index_tactile_2, origin xyz=0 0 0 rpy=0 0 0, axis 0 0 0
- added joint left_index_pad: type fixed, parent left_index_link_3, child left_index_pad, origin xyz=0.015999999999905 0.00779994490916784 0 rpy=0 0 0, axis 0 0 0
- added joint left_index_tip: type fixed, parent left_index_link_3, child left_index_tip, origin xyz=0.027999999999834 0 0 rpy=0 0 0, axis 0 0 0
- added joint left_middle_j0: type revolute, parent left_palm_link, child left_middle_link_0, origin xyz=0.0069979 -0.011496 0.1185 rpy=3.1416 -1.5708 0, axis 0 0 1, limit lower=-0.436 upper=0.436 effort=0 velocity=8.7266
- added joint left_middle_j1: type revolute, parent left_middle_link_0, child left_middle_link_1, origin xyz=0.016 0 0 rpy=1.5708 0 0, axis 0 0 1, limit lower=-0.349 upper=1.5708 effort=0 velocity=8.7266
- added joint left_middle_j1_sensor: type fixed, parent left_middle_link_1, child left_middle_tactile_0, origin xyz=0 0 0 rpy=0 0 0, axis 0 0 0
- added joint left_middle_j2: type revolute, parent left_middle_link_1, child left_middle_link_2, origin xyz=0.045 0 0 rpy=0 0 0, axis 0 0 1, limit lower=-0.0873 upper=1.745 effort=0 velocity=8.7266
- added joint left_middle_j2_sensor: type fixed, parent left_middle_link_2, child left_middle_tactile_1, origin xyz=0 0 0 rpy=0 0 0, axis 0 0 0
- added joint left_middle_j3: type revolute, parent left_middle_link_2, child left_middle_link_3, origin xyz=0.025 0 0 rpy=0 0 0, axis 0 0 1, limit lower=-0.0873 upper=1.745 effort=0 velocity=8.7266, mimic joint=left_middle_j2 multiplier=1.0 offset=0
- added joint left_middle_j3_sensor: type fixed, parent left_middle_link_3, child left_middle_tactile_2, origin xyz=0 0 0 rpy=0 0 0, axis 0 0 0
- added joint left_middle_pad: type fixed, parent left_middle_link_3, child left_middle_pad, origin xyz=0.0159999999999052 0.00789994490916761 0 rpy=0 0 0, axis 0 0 0
- added joint left_middle_tip: type fixed, parent left_middle_link_3, child left_middle_tip, origin xyz=0.0279999999998339 0 0 rpy=0 0 0, axis 0 0 0
- added joint left_pinky_j0: type revolute, parent left_palm_link, child left_pinky_link_0, origin xyz=0.0069979 0.034504 0.1125 rpy=3.1416 -1.5708 0, axis 0 0 1, limit lower=-0.436 upper=0.436 effort=0 velocity=8.7266
- added joint left_pinky_j1: type revolute, parent left_pinky_link_0, child left_pinky_link_1, origin xyz=0.016 0 0 rpy=1.5708 0 0, axis 0 0 1, limit lower=-0.349 upper=1.5708 effort=0 velocity=8.7266
- added joint left_pinky_j1_sensor: type fixed, parent left_pinky_link_1, child left_pinky_tactile_0, origin xyz=0 0 0 rpy=0 0 0, axis 0 0 0
- added joint left_pinky_j2: type revolute, parent left_pinky_link_1, child left_pinky_link_2, origin xyz=0.045 0 0 rpy=0 -4.2275E-05 0, axis 0 0 1, limit lower=-0.0873 upper=1.745 effort=0 velocity=8.7266
- added joint left_pinky_j2_sensor: type fixed, parent left_pinky_link_2, child left_pinky_tactile_1, origin xyz=0 0 0 rpy=0 0 0, axis 0 0 0
- added joint left_pinky_j3: type revolute, parent left_pinky_link_2, child left_pinky_link_3, origin xyz=0.025 0 0 rpy=0 0 0, axis 0 0 1, limit lower=-0.0873 upper=1.745 effort=0 velocity=8.7266, mimic joint=left_pinky_j2 multiplier=1.0 offset=0
- added joint left_pinky_j3_sensor: type fixed, parent left_pinky_link_3, child left_pinky_tactile_2, origin xyz=0 0 0 rpy=0 0 0, axis 0 0 0
- added joint left_pinky_pad: type fixed, parent left_pinky_link_3, child left_pinky_pad, origin xyz=0.0159999998319094 0.00789994490916776 0 rpy=0 4.22751595454715E-05 0, axis 0 0 0
- added joint left_pinky_tip: type fixed, parent left_pinky_link_3, child left_pinky_tip, origin xyz=0.0279999998211151 0 0 rpy=0 4.22751595454715E-05 0, axis 0 0 0
- added joint left_ring_j0: type revolute, parent left_palm_link, child left_ring_link_0, origin xyz=0.0069979 0.011503 0.1155 rpy=3.1416 -1.5708 0, axis 0 0 1, limit lower=-0.436 upper=0.436 effort=0 velocity=8.7266
- added joint left_ring_j1: type revolute, parent left_ring_link_0, child left_ring_link_1, origin xyz=0.016 0 0 rpy=1.5708 0 0, axis 0 0 1, limit lower=-0.349 upper=1.5708 effort=0 velocity=8.7266
- added joint left_ring_j1_sensor: type fixed, parent left_ring_link_1, child left_ring_tactile_0, origin xyz=0 0 0 rpy=0 0 0, axis 0 0 0
- added joint left_ring_j2: type revolute, parent left_ring_link_1, child left_ring_link_2, origin xyz=0.045 0 0 rpy=0 0 0, axis 0 0 1, limit lower=-0.0873 upper=1.745 effort=0 velocity=8.7266
- added joint left_ring_j2_sensor: type fixed, parent left_ring_link_2, child left_ring_tactile_1, origin xyz=0 0 0 rpy=0 0 0, axis 0 0 0
- added joint left_ring_j3: type revolute, parent left_ring_link_2, child left_ring_link_3, origin xyz=0.025 0 0 rpy=0 0 0, axis 0 0 1, limit lower=-0.0873 upper=1.745 effort=0 velocity=8.7266, mimic joint=left_ring_j2 multiplier=1.0 offset=0
- added joint left_ring_j3_sensor: type fixed, parent left_ring_link_3, child left_ring_tactile_2, origin xyz=0 0 0 rpy=0 0 0, axis 0 0 0
- added joint left_ring_pad: type fixed, parent left_ring_link_3, child left_ring_pad, origin xyz=0.015999999999905 0.00789994490916785 0 rpy=0 0 0, axis 0 0 0
- added joint left_ring_tip: type fixed, parent left_ring_link_3, child left_ring_tip, origin xyz=0.0279999999998339 0 0 rpy=0 0 0, axis 0 0 0
- added joint left_thumb_j0: type revolute, parent left_palm_link, child left_thumb_link_0, origin xyz=0.012998 -0.022996 0.0493 rpy=0 0 -1.5708, axis 0 0 1, limit lower=0 upper=1.3963 effort=0 velocity=8.7266
- added joint left_thumb_j1: type revolute, parent left_thumb_link_0, child left_thumb_link_1, origin xyz=0.0145 0 0 rpy=1.5708 0 -1.5708, axis 0 0 1, limit lower=-0.1745 upper=1.047 effort=0 velocity=8.7266
- added joint left_thumb_j2: type revolute, parent left_thumb_link_1, child left_thumb_link_2, origin xyz=0 0 -0.014 rpy=1.5708 0 1.5708, axis 0 0 1, limit lower=0 upper=1.396 effort=0 velocity=8.7266
- added joint left_thumb_j2_sensor: type fixed, parent left_thumb_link_2, child left_thumb_tactile_0, origin xyz=0 0 0 rpy=0 0 0, axis 0 0 0
- added joint left_thumb_j3: type revolute, parent left_thumb_link_2, child left_thumb_link_3, origin xyz=0 -0.055 0 rpy=0 0 -1.5708, axis 0 0 1, limit lower=-0.349 upper=1.396 effort=0 velocity=8.7266
- added joint left_thumb_j3_sensor: type fixed, parent left_thumb_link_3, child left_thumb_tactile_1, origin xyz=0 0 0 rpy=0 0 0, axis 0 0 0
- added joint left_thumb_j4: type revolute, parent left_thumb_link_3, child left_thumb_link_4, origin xyz=0.03 0 0 rpy=0 0 0, axis 0 0 1, limit lower=-0.349 upper=1.396 effort=0 velocity=8.7266, mimic joint=left_thumb_j3 multiplier=1.0 offset=0
- added joint left_thumb_j4_sensor: type fixed, parent left_thumb_link_4, child left_thumb_tactile_2, origin xyz=0 0 0 rpy=0 0 0, axis 0 0 0
- added joint left_thumb_pad: type fixed, parent left_thumb_link_4, child left_thumb_tip, origin xyz=0.028 0 0 rpy=0 0 0, axis 0 0 0
- added joint left_thumb_tip: type fixed, parent left_thumb_link_4, child left_thumb_pad, origin xyz=0.015 0.00779999999999999 0 rpy=0 0 0, axis 0 0 0
