Commit message: 1.修正URDF命名错误 2.添加LICENSE

File: apex_hand_right/apex_hand_right.urdf (robot description, URDF)
Before this commit: robot Apex_hand_right, 47 links, 46 joints
Links:
- removed link Palm_link_right
- removed link f0_link0
- removed link f0_link1
- removed link f0_link2
- removed link f0_link2sensor
- removed link f0_link3
- removed link f0_link3sensor
- removed link f0_link4
- removed link f0_link4sensor
- removed link f0_pad
- removed link f0_tip
- removed link f1_link0
- removed link f1_link1
- removed link f1_link1sensor
- removed link f1_link2
- removed link f1_link2sensor
- removed link f1_link3
- removed link f1_link3sensor
- removed link f1_pad
- removed link f1_tip
- removed link f2_link0
- removed link f2_link1
- removed link f2_link1sensor
- removed link f2_link2
- removed link f2_link2sensor
- removed link f2_link3
- removed link f2_link3sensor
- removed link f2_pad
- removed link f2_tip
- removed link f3_link0
- removed link f3_link1
- removed link f3_link1sensor
- removed link f3_link2
- removed link f3_link2sensor
- removed link f3_link3
- removed link f3_link3sensor
- removed link f3_pad
- removed link f3_tip
- removed link f4_link0
- removed link f4_link1
- removed link f4_link1sensor
- removed link f4_link2
- removed link f4_link2sensor
- removed link f4_link3
- removed link f4_link3sensor
- removed link f4_pad
- removed link f4_tip
- added link right_index_link_0, mass 0.0187941572496829; collision mesh filename=./meshes/right_index_link_0.STL; visual mesh filename=./meshes/right_index_link_0.STL
- added link right_index_link_1, mass 0.0290954766878931; collision mesh filename=./meshes/right_index_link_1.STL; visual mesh filename=./meshes/right_index_link_1.STL
- added link right_index_link_2, mass 0.0111427111396244; collision mesh filename=./meshes/right_index_link_2.STL; visual mesh filename=./meshes/right_index_link_2.STL
- added link right_index_link_3, mass 0.00518541203449776; collision mesh filename=./meshes/right_index_link_3.STL; visual mesh filename=./meshes/right_index_link_3.STL
- added link right_index_pad, mass 8.20481262582146E-06; collision mesh filename=./meshes/right_index_pad.STL; visual mesh filename=./meshes/right_index_pad.STL
- added link right_index_tactile_0, mass 0.00892665816512101; collision mesh filename=./meshes/right_index_tactile_0.STL; visual mesh filename=./meshes/right_index_tactile_0.STL
- added link right_index_tactile_1, mass 0.00363566690918231; collision mesh filename=./meshes/right_index_tactile_1.STL; visual mesh filename=./meshes/right_index_tactile_1.STL
- added link right_index_tactile_2, mass 0.00986650294125371; collision mesh filename=./meshes/right_index_tactile_2.STL; visual mesh filename=./meshes/right_index_tactile_2.STL
- added link right_index_tip, mass 8.20481262582146E-06; collision mesh filename=./meshes/right_index_tip.STL; visual mesh filename=./meshes/right_index_tip.STL
- added link right_middle_link_0, mass 0.0187941572496829; collision mesh filename=./meshes/right_middle_link_0.STL; visual mesh filename=./meshes/right_middle_link_0.STL
- added link right_middle_link_1, mass 0.0290954766874994; collision mesh filename=./meshes/right_middle_link_1.STL; visual mesh filename=./meshes/right_middle_link_1.STL
- added link right_middle_link_2, mass 0.0111427111396243; collision mesh filename=./meshes/right_middle_link_2.STL; visual mesh filename=./meshes/right_middle_link_2.STL
- added link right_middle_link_3, mass 0.00518541203449776; collision mesh filename=./meshes/right_middle_link_3.STL; visual mesh filename=./meshes/right_middle_link_3.STL
- added link right_middle_pad, mass 8.20481262582145E-06; collision mesh filename=./meshes/right_middle_pad.STL; visual mesh filename=./meshes/right_middle_pad.STL
- added link right_middle_tactile_0, mass 0.00892666891987732; collision mesh filename=./meshes/right_middle_tactile_0.STL; visual mesh filename=./meshes/right_middle_tactile_0.STL
- added link right_middle_tactile_1, mass 0.00363566690918773; collision mesh filename=./meshes/right_middle_tactile_1.STL; visual mesh filename=./meshes/right_middle_tactile_1.STL
- added link right_middle_tactile_2, mass 0.00986650306941366; collision mesh filename=./meshes/right_middle_tactile_2.STL; visual mesh filename=./meshes/right_middle_tactile_2.STL
- added link right_middle_tip, mass 8.20481262582146E-06; collision mesh filename=./meshes/right_middle_tip.STL; visual mesh filename=./meshes/right_middle_tip.STL
- added link right_palm_link, mass 0.262735816921321; collision mesh filename=./meshes/right_palm_link.STL; visual mesh filename=./meshes/right_palm_link.STL
- added link right_pinky_link_0, mass 0.0187941572496829; collision mesh filename=./meshes/right_pinky_link_0.STL; visual mesh filename=./meshes/right_pinky_link_0.STL
- added link right_pinky_link_1, mass 0.0290954766874994; collision mesh filename=./meshes/right_pinky_link_1.STL; visual mesh filename=./meshes/right_pinky_link_1.STL
- added link right_pinky_link_2, mass 0.0111427111396244; collision mesh filename=./meshes/right_pinky_link_2.STL; visual mesh filename=./meshes/right_pinky_link_2.STL
- added link right_pinky_link_3, mass 0.00518541203449776; collision mesh filename=./meshes/right_pinky_link_3.STL; visual mesh filename=./meshes/right_pinky_link_3.STL
- added link right_pinky_pad, mass 8.20481262582142E-06; collision mesh filename=./meshes/right_pinky_pad.STL; visual mesh filename=./meshes/right_pinky_pad.STL
- added link right_pinky_tactile_0, mass 0.00892665816501502; collision mesh filename=./meshes/right_pinky_tactile_0.STL; visual mesh filename=./meshes/right_pinky_tactile_0.STL
- added link right_pinky_tactile_1, mass 0.00363566688942038; collision mesh filename=./meshes/right_pinky_tactile_1.STL; visual mesh filename=./meshes/right_pinky_tactile_1.STL
- added link right_pinky_tactile_2, mass 0.0098665026793508; collision mesh filename=./meshes/right_pinky_tactile_2.STL; visual mesh filename=./meshes/right_pinky_tactile_2.STL
- added link right_pinky_tip, mass 8.20481262582146E-06; collision mesh filename=./meshes/right_pinky_tip.STL; visual mesh filename=./meshes/right_pinky_tip.STL
- added link right_ring_link_0, mass 0.0187941572496829; collision mesh filename=./meshes/right_ring_link_0.STL; visual mesh filename=./meshes/right_ring_link_0.STL
- added link right_ring_link_1, mass 0.0290954766872578; collision mesh filename=./meshes/right_ring_link_1.STL; visual mesh filename=./meshes/right_ring_link_1.STL
- added link right_ring_link_2, mass 0.0111427111396244; collision mesh filename=./meshes/right_ring_link_2.STL; visual mesh filename=./meshes/right_ring_link_2.STL
- added link right_ring_link_3, mass 0.00518541203449777; collision mesh filename=./meshes/right_ring_link_3.STL; visual mesh filename=./meshes/right_ring_link_3.STL
- added link right_ring_pad, mass 8.20481262582145E-06; collision mesh filename=./meshes/right_ring_pad.STL; visual mesh filename=./meshes/right_ring_pad.STL
- added link right_ring_tactile_0, mass 0.0089266622621125; collision mesh filename=./meshes/right_ring_tactile_0.STL; visual mesh filename=./meshes/right_ring_tactile_0.STL
- added link right_ring_tactile_1, mass 0.00363566684156878; collision mesh filename=./meshes/right_ring_tactile_1.STL; visual mesh filename=./meshes/right_ring_tactile_1.STL
- added link right_ring_tactile_2, mass 0.00986650304596387; collision mesh filename=./meshes/right_ring_tactile_2.STL; visual mesh filename=./meshes/right_ring_tactile_2.STL
- added link right_ring_tip, mass 8.20481262582144E-06; collision mesh filename=./meshes/right_ring_tip.STL; visual mesh filename=./meshes/right_ring_tip.STL
- added link right_thumb_link_0, mass 0.0109675846438251; collision mesh filename=./meshes/right_thumb_link_0.STL; visual mesh filename=./meshes/right_thumb_link_0.STL
- added link right_thumb_link_1, mass 0.015512035165475; collision mesh filename=./meshes/right_thumb_link_1.STL; visual mesh filename=./meshes/right_thumb_link_1.STL
- added link right_thumb_link_2, mass 0.0478768695058164; collision mesh filename=./meshes/right_thumb_link_2.STL; visual mesh filename=./meshes/right_thumb_link_2.STL
- added link right_thumb_link_3, mass 0.020327269172061; collision mesh filename=./meshes/right_thumb_link_3.STL; visual mesh filename=./meshes/right_thumb_link_3.STL
- added link right_thumb_link_4, mass 0.00936725934380467; collision mesh filename=./meshes/right_thumb_link_4.STL; visual mesh filename=./meshes/right_thumb_link_4.STL
- added link right_thumb_pad, mass 8.20481262582145E-06; collision mesh filename=./meshes/right_thumb_pad.STL; visual mesh filename=./meshes/right_thumb_pad.STL
- added link right_thumb_tactile_0, mass 0.0359955797573235; collision mesh filename=./meshes/right_thumb_tactile_0.STL; visual mesh filename=./meshes/right_thumb_tactile_0.STL
- added link right_thumb_tactile_1, mass 0.00938453614062146; collision mesh filename=./meshes/right_thumb_tactile_1.STL; visual mesh filename=./meshes/right_thumb_tactile_1.STL
- added link right_thumb_tactile_2, mass 0.00986648442645367; collision mesh filename=./meshes/right_thumb_tactile_2.STL; visual mesh filename=./meshes/right_thumb_tactile_2.STL
- added link right_thumb_tip, mass 8.20481262582145E-06; collision mesh filename=./meshes/right_thumb_tip.STL; visual mesh filename=./meshes/right_thumb_tip.STL
Joints:
- removed joint f0_joint0
- removed joint f0_joint1
- removed joint f0_joint2
- removed joint f0_joint2sensor
- removed joint f0_joint3
- removed joint f0_joint3sensor
- removed joint f0_joint4
- removed joint f0_joint4sensor
- removed joint f0_pad
- removed joint f0_tip
- removed joint f1_joint0
- removed joint f1_joint1
- removed joint f1_joint1sensor
- removed joint f1_joint2
- removed joint f1_joint2sensor
- removed joint f1_joint3
- removed joint f1_joint3sensor
- removed joint f1_pad
- removed joint f1_tip
- removed joint f2_joint0
- removed joint f2_joint1
- removed joint f2_joint1sensor
- removed joint f2_joint2
- removed joint f2_joint2sensor
- removed joint f2_joint3
- removed joint f2_joint3sensor
- removed joint f2_pad
- removed joint f2_tip
- removed joint f3_joint0
- removed joint f3_joint1
- removed joint f3_joint2
- removed joint f3_joint2sensor
- removed joint f3_joint3
- removed joint f3_joint3sensor
- removed joint f3_link1sensor
- removed joint f3_pad
- removed joint f3_tip
- removed joint f4_joint0
- removed joint f4_joint1
- removed joint f4_joint1sensor
- removed joint f4_joint2
- removed joint f4_joint3
- removed joint f4_joint3sensor
- removed joint f4_link2sensor
- removed joint f4_pad
- removed joint f4_tip
- added joint right_index_j0: type revolute, parent right_palm_link, child right_index_link_0, origin xyz=0.0069979 0.034496 0.1155 rpy=0 -1.5708 0, axis 0 0 1, limit lower=-0.436 upper=0.436 effort=0 velocity=8.7266
- added joint right_index_j1: type revolute, parent right_index_link_0, child right_index_link_1, origin xyz=0.016 0 0 rpy=-1.570795877559 0 0, axis 0 0 1, limit lower=-0.349 upper=1.5708 effort=0 velocity=8.7266
- added joint right_index_j1_sensor: type fixed, parent right_index_link_1, child right_index_tactile_0, origin xyz=0 0 0 rpy=0 0 0, axis 0 0 0
- added joint right_index_j2: type revolute, parent right_index_link_1, child right_index_link_2, origin xyz=0.045 0 0 rpy=0 0 0, axis 0 0 1, limit lower=-0.0873 upper=1.745 effort=0 velocity=8.7266
- added joint right_index_j2_sensor: type fixed, parent right_index_link_2, child right_index_tactile_1, origin xyz=0 0 0 rpy=0 0 0, axis 0 0 0, limit lower=0 upper=0 effort=0 velocity=8.7266
- added joint right_index_j3: type revolute, parent right_index_link_2, child right_index_link_3, origin xyz=0.025 0 0 rpy=0 0 0, axis 0 0 1, limit lower=-0.0873 upper=1.745 effort=0 velocity=8.7266, mimic joint=right_index_j2 multiplier=1.0 offset=0
- added joint right_index_j3_sensor: type fixed, parent right_index_link_3, child right_index_tactile_2, origin xyz=0 0 0 rpy=0 0 0, axis 0 0 0
- added joint right_index_pad: type fixed, parent right_index_link_3, child right_index_pad, origin xyz=0.016 0.00789999999999919 0 rpy=0 0 0, axis 0 0 0
- added joint right_index_tip: type fixed, parent right_index_link_3, child right_index_tip, origin xyz=0.028 0 0 rpy=0 0 0, axis 0 0 0
- added joint right_middle_j0: type revolute, parent right_palm_link, child right_middle_link_0, origin xyz=0.0069979 0.011496 0.1185 rpy=0 -1.5708 0, axis 0 0 1, limit lower=-0.436 upper=0.436 effort=0 velocity=8.7266
- added joint right_middle_j1: type revolute, parent right_middle_link_0, child right_middle_link_1, origin xyz=0.016 0 0 rpy=-1.5708 0 0, axis 0 0 1, limit lower=-0.349 upper=1.5708 effort=0 velocity=8.7266
- added joint right_middle_j1_sensor: type fixed, parent right_middle_link_1, child right_middle_tactile_0, origin xyz=0 0 0 rpy=0 0 0, axis 0 0 0
- added joint right_middle_j2: type revolute, parent right_middle_link_1, child right_middle_link_2, origin xyz=0.045 0 0 rpy=0 0 -0.0004769, axis 0 0 1, limit lower=-0.0873 upper=1.745 effort=0 velocity=8.7266
- added joint right_middle_j2_sensor: type fixed, parent right_middle_link_2, child right_middle_tactile_1, origin xyz=0 0 0 rpy=0 0 0, axis 0 0 0
- added joint right_middle_j3: type revolute, parent right_middle_link_2, child right_middle_link_3, origin xyz=0.025 1.1923E-05 0 rpy=0 0 0.0004769, axis 0 0 1, limit lower=-0.0873 upper=1.745 effort=0 velocity=8.7266, mimic joint=right_middle_j2 multiplier=1.0 offset=0
- added joint right_middle_j3_sensor: type fixed, parent right_middle_link_3, child right_middle_tactile_2, origin xyz=0 0 0 rpy=0 0 0, axis 0 0 0
- added joint right_middle_pad: type fixed, parent right_middle_link_3, child right_middle_pad, origin xyz=0.0160000000000002 0.00789999999999927 0 rpy=0 0 0, axis 0 0 0
- added joint right_middle_tip: type fixed, parent right_middle_link_3, child right_middle_tip, origin xyz=0.0280000000000001 0 0 rpy=0 0 0, axis 0 0 0
- added joint right_pinky_j0: type revolute, parent right_palm_link, child right_pinky_link_0, origin xyz=0.0069979 -0.034504 0.1125 rpy=0 -1.5708 0, axis 0 0 1, limit lower=-0.436 upper=0.436 effort=0 velocity=8.7266
- added joint right_pinky_j1: type revolute, parent right_pinky_link_0, child right_pinky_link_1, origin xyz=0.016 0 0 rpy=-1.5708 0 0, axis 0 0 1, limit lower=-0.349 upper=1.5708 effort=0 velocity=8.7266
- added joint right_pinky_j1_sensor: type fixed, parent right_pinky_link_1, child right_pinky_tactile_0, origin xyz=0 0 0 rpy=0 0 0, axis 0 0 0
- added joint right_pinky_j2: type revolute, parent right_pinky_link_1, child right_pinky_link_2, origin xyz=0.045 0 0 rpy=0 0 -0.0004769, axis 0 0 1, limit lower=-0.0873 upper=1.745 effort=0 velocity=8.7266
- added joint right_pinky_j3: type revolute, parent right_pinky_link_2, child right_pinky_link_3, origin xyz=0.025 1.1923E-05 0 rpy=0 0 0, axis 0 0 1, limit lower=-0.0873 upper=1.745 effort=0 velocity=8.7266, mimic joint=right_pinky_j2 multiplier=1.0 offset=0
- added joint right_pinky_j3_sensor: type fixed, parent right_pinky_link_3, child right_pinky_tactile_2, origin xyz=0 0 0 rpy=0 0 0, axis 0 0 0
- added joint right_pinky_pad: type fixed, parent right_pinky_link_3, child right_pinky_pad, origin xyz=0.0159962306453115 0.00790762955265271 0 rpy=0 0 0.000476903207341931, axis 0 0 0
- added joint right_pinky_tactile_1: type fixed, parent right_pinky_link_2, child right_pinky_tactile_1, origin xyz=0 0 0 rpy=0 0 0, axis 0 0 0
- added joint right_pinky_tip: type fixed, parent right_pinky_link_3, child right_pinky_tip, origin xyz=0.0279999968158867 1.33532892995824E-05 0 rpy=0 0 0.000476903207341931, axis 0 0 0
- added joint right_ring_j0: type revolute, parent right_palm_link, child right_ring_link_0, origin xyz=0.0069979 -0.011503 0.1155 rpy=0 -1.5708 0, axis 0 0 1, limit lower=-0.436 upper=0.436 effort=0 velocity=8.7266
- added joint right_ring_j1: type revolute, parent right_ring_link_0, child right_ring_link_1, origin xyz=0.016 0 0 rpy=-1.5708 -0.0004769 0, axis 0 0 1, limit lower=-0.349 upper=1.5708 effort=0 velocity=8.7266
- added joint right_ring_j2: type revolute, parent right_ring_link_1, child right_ring_link_2, origin xyz=0.045 2.1461E-05 0 rpy=0 0 0.0004769, axis 0 0 1, limit lower=-0.0873 upper=1.745 effort=0 velocity=8.7266
- added joint right_ring_j2_sensor: type fixed, parent right_ring_link_2, child right_ring_tactile_1, origin xyz=0 0 0 rpy=0 0 0, axis 0 0 0
- added joint right_ring_j3: type revolute, parent right_ring_link_2, child right_ring_link_3, origin xyz=0.025 0 0 rpy=0 0 0, axis 0 0 1, limit lower=-0.0873 upper=1.745 effort=0 velocity=8.7266, mimic joint=right_ring_j2 multiplier=1.0 offset=0
- added joint right_ring_j3_sensor: type fixed, parent right_ring_link_3, child right_ring_tactile_2, origin xyz=0 0 0 rpy=0 0 0, axis 0 0 0
- added joint right_ring_pad: type fixed, parent right_ring_link_3, child right_ring_pad, origin xyz=0.016 0.0078999999999992 0 rpy=0 0 -0.000476903207335163, axis 0 0 0
- added joint right_ring_tactile_0: type fixed, parent right_ring_link_1, child right_ring_tactile_0, origin xyz=0 0 0 rpy=0 0 0, axis 0 0 0
- added joint right_ring_tip: type fixed, parent right_ring_link_3, child right_ring_tip, origin xyz=0.028 0 0 rpy=0 0 -0.000476903207335163, axis 0 0 0
- added joint right_thumb_j0: type revolute, parent right_palm_link, child right_thumb_link_0, origin xyz=0.012998 0.022996 0.0493 rpy=3.1416 0 1.5708, axis 0 0 1, limit lower=0 upper=1.3963 effort=0 velocity=8.7266
- added joint right_thumb_j1: type revolute, parent right_thumb_link_0, child right_thumb_link_1, origin xyz=0.0145 0 0 rpy=-1.5708 0 -1.5708, axis 0 0 1, limit lower=-0.1745 upper=1.047 effort=0 velocity=8.7266
- added joint right_thumb_j2: type revolute, parent right_thumb_link_1, child right_thumb_link_2, origin xyz=0 0 0.014 rpy=-1.5708 0 1.5708, axis 0 0 1, limit lower=0 upper=1.396 effort=0 velocity=8.7266
- added joint right_thumb_j2_sensor: type fixed, parent right_thumb_link_2, child right_thumb_tactile_0, origin xyz=0 0 0 rpy=0 0 0, axis 0 0 0
- added joint right_thumb_j3: type revolute, parent right_thumb_link_2, child right_thumb_link_3, origin xyz=0 -0.055 0 rpy=0 0 -1.5708, axis 0 0 1, limit lower=-0.349 upper=1.396 effort=0 velocity=8.7266
- added joint right_thumb_j3_sensor: type fixed, parent right_thumb_link_3, child right_thumb_tactile_1, origin xyz=0 0 0 rpy=0 0 0, axis 0 0 0
- added joint right_thumb_j4: type revolute, parent right_thumb_link_3, child right_thumb_link_4, origin xyz=0.03 0 0 rpy=0 0 0, axis 0 0 1, limit lower=-0.349 upper=1.396 effort=0 velocity=8.7266, mimic joint=right_thumb_j3 multiplier=1.0 offset=0
- added joint right_thumb_j4_sensor: type fixed, parent right_thumb_link_4, child right_thumb_tactile_2, origin xyz=0 0 0 rpy=0 0 0, axis 0 0 0
- added joint right_thumb_pad: type fixed, parent right_thumb_link_4, child right_thumb_pad, origin xyz=0.015 0.00779999999999999 0 rpy=0 0 0, axis 0 0 0
- added joint right_thumb_tip: type fixed, parent right_thumb_link_4, child right_thumb_tip, origin xyz=0.028 0 0 rpy=0 0 0, axis 0 0 0
