Commit message: Updated URDF files for new ApexHand version

File: apex_hand_left/apex_hand_left.urdf (robot description, URDF)
Before this commit: robot left_apex_hand, 47 links, 46 joints
Links:
- removed link left_index_link_0
- removed link left_index_link_1
- removed link left_index_link_2
- removed link left_index_link_3
- removed link left_index_tactile_0
- removed link left_index_tactile_1
- removed link left_index_tactile_2
- removed link left_middle_link_0
- removed link left_middle_link_1
- removed link left_middle_link_2
- removed link left_middle_link_3
- removed link left_middle_tactile_0
- removed link left_middle_tactile_1
- removed link left_middle_tactile_2
- removed link left_pinky_link_0
- removed link left_pinky_link_1
- removed link left_pinky_link_2
- removed link left_pinky_link_3
- removed link left_pinky_tactile_0
- removed link left_pinky_tactile_1
- removed link left_pinky_tactile_2
- removed link left_ring_link_0
- removed link left_ring_link_1
- removed link left_ring_link_2
- removed link left_ring_link_3
- removed link left_ring_tactile_0
- removed link left_ring_tactile_1
- removed link left_ring_tactile_2
- removed link left_thumb_link_0
- removed link left_thumb_link_1
- removed link left_thumb_link_2
- removed link left_thumb_link_3
- removed link left_thumb_link_4
- removed link left_thumb_tactile_0
- removed link left_thumb_tactile_1
- removed link left_thumb_tactile_2
- added link left_index_link0, mass 0.018794; collision mesh filename=./meshes/left_index_link0.STL; visual mesh filename=./meshes/left_index_link0.STL
- added link left_index_link1, mass 0.029095; collision mesh filename=./meshes/left_index_link1.STL; visual mesh filename=./meshes/left_index_link1.STL
- added link left_index_link2, mass 0.011142; collision mesh filename=./meshes/left_index_link2.STL; visual mesh filename=./meshes/left_index_link2.STL
- added link left_index_link3, mass 0.005232; collision mesh filename=./meshes/left_index_link3.STL; visual mesh filename=./meshes/left_index_link3.STL
- added link left_index_tactile0, mass 0.008926; collision mesh filename=./meshes/left_index_tactile0.STL; visual mesh filename=./meshes/left_index_tactile0.STL
- added link left_index_tactile1, mass 0.003635; collision mesh filename=./meshes/left_index_tactile1.STL; visual mesh filename=./meshes/left_index_tactile1.STL
- added link left_index_tactile2, mass 0.009866; collision mesh filename=./meshes/left_index_tactile2.STL; visual mesh filename=./meshes/left_index_tactile2.STL
- added link left_middle_link0, mass 0.018794; collision mesh filename=./meshes/left_middle_link0.STL; visual mesh filename=./meshes/left_middle_link0.STL
- added link left_middle_link1, mass 0.029095; collision mesh filename=./meshes/left_middle_link1.STL; visual mesh filename=./meshes/left_middle_link1.STL
- added link left_middle_link2, mass 0.011142; collision mesh filename=./meshes/left_middle_link2.STL; visual mesh filename=./meshes/left_middle_link2.STL
- added link left_middle_link3, mass 0.005232; collision mesh filename=./meshes/left_middle_link3.STL; visual mesh filename=./meshes/left_middle_link3.STL
- added link left_middle_tactile0, mass 0.008926; collision mesh filename=./meshes/left_middle_tactile0.STL; visual mesh filename=./meshes/left_middle_tactile0.STL
- added link left_middle_tactile1, mass 0.003635; collision mesh filename=./meshes/left_middle_tactile1.STL; visual mesh filename=./meshes/left_middle_tactile1.STL
- added link left_middle_tactile2, mass 0.009866; collision mesh filename=./meshes/left_middle_tactile2.STL; visual mesh filename=./meshes/left_middle_tactile2.STL
- added link left_palm_base, mass 0.1; collision mesh filename=./meshes/left_palm_base.STL; visual mesh filename=./meshes/left_palm_base.STL
- added link left_palm_tactile, mass 0; collision mesh filename=./meshes/left_palm_tactile.STL; visual mesh filename=./meshes/left_palm_tactile.STL
- added link left_pinky_link0, mass 0.018794; collision mesh filename=./meshes/left_pinky_link0.STL; visual mesh filename=./meshes/left_pinky_link0.STL
- added link left_pinky_link1, mass 0.029095; collision mesh filename=./meshes/left_pinky_link1.STL; visual mesh filename=./meshes/left_pinky_link1.STL
- added link left_pinky_link2, mass 0.011142; collision mesh filename=./meshes/left_pinky_link2.STL; visual mesh filename=./meshes/left_pinky_link2.STL
- added link left_pinky_link3, mass 0.005232; collision mesh filename=./meshes/left_pinky_link3.STL; visual mesh filename=./meshes/left_pinky_link3.STL
- added link left_pinky_tactile0, mass 0.008926; collision mesh filename=./meshes/left_pinky_tactile0.STL; visual mesh filename=./meshes/left_pinky_tactile0.STL
- added link left_pinky_tactile1, mass 0.003635; collision mesh filename=./meshes/left_pinky_tactile1.STL; visual mesh filename=./meshes/left_pinky_tactile1.STL
- added link left_pinky_tactile2, mass 0.009866; collision mesh filename=./meshes/left_pinky_tactile2.STL; visual mesh filename=./meshes/left_pinky_tactile2.STL
- added link left_ring_link0, mass 0.018794; collision mesh filename=./meshes/left_ring_link0.STL; visual mesh filename=./meshes/left_ring_link0.STL
- added link left_ring_link1, mass 0.029095; collision mesh filename=./meshes/left_ring_link1.STL; visual mesh filename=./meshes/left_ring_link1.STL
- added link left_ring_link2, mass 0.011142; collision mesh filename=./meshes/left_ring_link2.STL; visual mesh filename=./meshes/left_ring_link2.STL
- added link left_ring_link3, mass 0.005232; collision mesh filename=./meshes/left_ring_link3.STL; visual mesh filename=./meshes/left_ring_link3.STL
- added link left_ring_tactile0, mass 0.008926; collision mesh filename=./meshes/left_ring_tactile0.STL; visual mesh filename=./meshes/left_ring_tactile0.STL
- added link left_ring_tactile1, mass 0.003635; collision mesh filename=./meshes/left_ring_tactile1.STL; visual mesh filename=./meshes/left_ring_tactile1.STL
- added link left_ring_tactile2, mass 0.009866; collision mesh filename=./meshes/left_ring_tactile2.STL; visual mesh filename=./meshes/left_ring_tactile2.STL
- added link left_thumb_link0, mass 0.010968; collision mesh filename=./meshes/left_thumb_link0.STL; visual mesh filename=./meshes/left_thumb_link0.STL
- added link left_thumb_link1, mass 0.01551203; collision mesh filename=./meshes/left_thumb_link1.STL; visual mesh filename=./meshes/left_thumb_link1.STL
- added link left_thumb_link2, mass 0.032423; collision mesh filename=./meshes/left_thumb_link2.STL; visual mesh filename=./meshes/left_thumb_link2.STL
- added link left_thumb_link3, mass 0.018383721; collision mesh filename=./meshes/left_thumb_link3.STL; visual mesh filename=./meshes/left_thumb_link3.STL
- added link left_thumb_link4, mass 0.007655847; collision mesh filename=./meshes/left_thumb_link4.STL; visual mesh filename=./meshes/left_thumb_link4.STL
- added link left_thumb_tactile0, mass 0.035996; collision mesh filename=./meshes/left_thumb_tactile0.STL; visual mesh filename=./meshes/left_thumb_tactile0.STL
- added link left_thumb_tactile1, mass 0.0093845; collision mesh filename=./meshes/left_thumb_tactile1.STL; visual mesh filename=./meshes/left_thumb_tactile1.STL
- added link left_thumb_tactile2, mass 0.0098665; collision mesh filename=./meshes/left_thumb_tactile2.STL; visual mesh filename=./meshes/left_thumb_tactile2.STL
- link left_index_pad: mass 8.20481262582146E-06 -> 7.854E-07
- link left_index_tip: mass 8.20481262582146E-06 -> 9.8175E-08
- link left_middle_pad: mass 8.20481262582145E-06 -> 7.854E-07
- link left_middle_tip: mass 8.20481262582144E-06 -> 9.8175E-08
- link left_palm_link: mass 0.262853650060054 -> 0.2
- link left_pinky_pad: mass 8.20481262582147E-06 -> 7.854E-07
- link left_pinky_tip: mass 8.20481262582144E-06 -> 9.8175E-08
- link left_ring_pad: mass 8.20481262582145E-06 -> 7.854E-07
- link left_ring_tip: mass 8.20481262582146E-06 -> 9.8175E-08
- link left_thumb_pad: mass 8.20481262582145E-06 -> 7.854E-07
- link left_thumb_tip: mass 8.20481262582146E-06 -> 9.8175E-08
Joints:
- removed joint left_index_j1_sensor
- removed joint left_index_j2_sensor
- removed joint left_index_j3_sensor
- removed joint left_index_pad
- removed joint left_index_tip
- removed joint left_middle_j1_sensor
- removed joint left_middle_j2_sensor
- removed joint left_middle_j3_sensor
- removed joint left_middle_pad
- removed joint left_middle_tip
- removed joint left_pinky_j1_sensor
- removed joint left_pinky_j2_sensor
- removed joint left_pinky_j3_sensor
- removed joint left_pinky_pad
- removed joint left_pinky_tip
- removed joint left_ring_j1_sensor
- removed joint left_ring_j2_sensor
- removed joint left_ring_j3_sensor
- removed joint left_ring_pad
- removed joint left_ring_tip
- removed joint left_thumb_j2_sensor
- removed joint left_thumb_j3_sensor
- removed joint left_thumb_j4_sensor
- removed joint left_thumb_pad
- removed joint left_thumb_tip
- added joint left_index_pad_fix: type fixed, parent left_index_tactile2, child left_index_pad, origin xyz=0.0170961447591369 0.00719554486026085 -0.000496366780427283 rpy=0 0 0, axis 0 0 0
- added joint left_index_tactile0_fix: type fixed, parent left_index_link1, child left_index_tactile0, origin xyz=0 0 0 rpy=0 0 0, axis 0 0 0
- added joint left_index_tactile1_fix: type fixed, parent left_index_link2, child left_index_tactile1, origin xyz=0 0 0 rpy=0 0 0, axis 0 0 0
- added joint left_index_tactile2_fix: type fixed, parent left_index_link3, child left_index_tactile2, origin xyz=0 0 0 rpy=0 0 0, axis 0 0 0
- added joint left_index_tip_fix: type fixed, parent left_index_tactile2, child left_index_tip, origin xyz=0.0276721667197929 0.000550277924151174 -0.000246366780427262 rpy=0 0 0, axis 0 0 0
- added joint left_middle_pad_fix: type fixed, parent left_middle_tactile2, child left_middle_pad, origin xyz=0.017096144759137 0.00719554486026086 -0.000496366780427282 rpy=0 0 0, axis 0 0 0
- added joint left_middle_tactile0_fix: type fixed, parent left_middle_link1, child left_middle_tactile0, origin xyz=0 0 0 rpy=0 0 0, axis 0 0 0
- added joint left_middle_tactile1_fix: type fixed, parent left_middle_link2, child left_middle_tactile1, origin xyz=0 0 0 rpy=0 0 0, axis 0 0 0
- added joint left_middle_tactile2_fix: type fixed, parent left_middle_link3, child left_middle_tactile2, origin xyz=0 0 0 rpy=0 0 0, axis 0 0 0
- added joint left_middle_tip_fix: type fixed, parent left_middle_tactile2, child left_middle_tip, origin xyz=0.027672166719793 0.000550277924151176 -0.00024636678042729 rpy=0 0 0, axis 0 0 0
- added joint left_palm_base_fix: type fixed, parent left_palm_link, child left_palm_base, origin xyz=0 0 0 rpy=0 0 0, axis 0 0 0
- added joint left_palm_tactile_fix: type fixed, parent left_palm_link, child left_palm_tactile, origin xyz=0 0 0 rpy=0 0 0, axis 0 0 0
- added joint left_pinky_pad_fix: type fixed, parent left_pinky_tactile2, child left_pinky_pad, origin xyz=0.017096 0.0071955 -0.00049637 rpy=0 0 0, axis 0 0 0
- added joint left_pinky_tactile0_fix: type fixed, parent left_pinky_link1, child left_pinky_tactile0, origin xyz=0 0 0 rpy=0 0 0, axis 0 0 0
- added joint left_pinky_tactile1_fix: type fixed, parent left_pinky_link2, child left_pinky_tactile1, origin xyz=0 0 0 rpy=0 0 0, axis 0 0 0
- added joint left_pinky_tactile2_fix: type fixed, parent left_pinky_link3, child left_pinky_tactile2, origin xyz=0 0 0 rpy=0 0 0, axis 0 0 0
- added joint left_pinky_tip_fix: type fixed, parent left_pinky_tactile2, child left_pinky_tip, origin xyz=0.027672 0.00055028 -0.00024637 rpy=0 0 0, axis 0 0 0
- added joint left_ring_pad_fix: type fixed, parent left_ring_tactile2, child left_ring_pad, origin xyz=0.017096144759137 0.00719554486026086 -0.000496366780427282 rpy=0 0 0, axis 0 0 0
- added joint left_ring_tactile0_fix: type fixed, parent left_ring_link1, child left_ring_tactile0, origin xyz=0 0 0 rpy=0 0 0, axis 0 0 0
- added joint left_ring_tactile1_fix: type fixed, parent left_ring_link2, child left_ring_tactile1, origin xyz=0 0 0 rpy=0 0 0, axis 0 0 0
- added joint left_ring_tactile2_fix: type fixed, parent left_ring_link3, child left_ring_tactile2, origin xyz=0 0 0 rpy=0 0 0, axis 0 0 0
- added joint left_ring_tip_fix: type fixed, parent left_ring_tactile2, child left_ring_tip, origin xyz=0.027672166719793 0.000550277924151177 -0.000246366780427318 rpy=0 0 0, axis 0 0 0
- added joint left_thumb_pad_fix: type fixed, parent left_thumb_tactile2, child left_thumb_pad, origin xyz=0.018471 0.0088124 0 rpy=0 0 0, axis 0 0 0
- added joint left_thumb_tactile0_fix: type fixed, parent left_thumb_link2, child left_thumb_tactile0, origin xyz=0 0 0 rpy=0 0 0, axis 0 0 0
- added joint left_thumb_tactile1_fix: type fixed, parent left_thumb_link3, child left_thumb_tactile1, origin xyz=0 0 0 rpy=0 0 0, axis 0 0 0
- added joint left_thumb_tactile2_fix: type fixed, parent left_thumb_link4, child left_thumb_tactile2, origin xyz=0 0 0 rpy=0 0 0, axis 0 0 0
- added joint left_thumb_tip_fix: type fixed, parent left_thumb_tactile2, child left_thumb_tip, origin xyz=0.029863 -0.00039744 0 rpy=0 0 0, axis 0 0 0
- joint left_index_j0: child left_index_link_0 -> left_index_link0; limit lower=-0.436 upper=0.436 effort=0 velocity=8.7266 -> lower=-0.4363 upper=0.4363 effort=0 velocity=0; origin xyz=0.0069979 -0.034496 0.1155 rpy=3.1416 -1.5708 0 -> xyz=0.0071 -0.034496 0.1188 rpy=0 -1.5708 3.1416; parent left_palm_link -> left_palm_base
- joint left_index_j1: child left_index_link_1 -> left_index_link1; limit lower=-0.349 upper=1.5708 effort=0 velocity=8.7266 -> lower=-0.349 upper=1.5707 effort=0 velocity=0; parent left_index_link_0 -> left_index_link0
- joint left_index_j2: child left_index_link_2 -> left_index_link2; limit lower=-0.0873 upper=1.745 effort=0 velocity=8.7266 -> lower=-0.0872 upper=1.7453 effort=0 velocity=0; parent left_index_link_1 -> left_index_link1
- joint left_index_j3: child left_index_link_3 -> left_index_link3; limit lower=-0.0873 upper=1.745 effort=0 velocity=8.7266 -> lower=-0.0872 upper=1.7453 effort=0 velocity=0; parent left_index_link_2 -> left_index_link2
- joint left_middle_j0: child left_middle_link_0 -> left_middle_link0; limit lower=-0.436 upper=0.436 effort=0 velocity=8.7266 -> lower=-0.4363 upper=0.4363 effort=0 velocity=0; origin xyz=0.0069979 -0.011496 0.1185 rpy=3.1416 -1.5708 0 -> xyz=0.0071 -0.011496 0.1218 rpy=0 -1.5708 3.1416; parent left_palm_link -> left_palm_base
- joint left_middle_j1: child left_middle_link_1 -> left_middle_link1; limit lower=-0.349 upper=1.5708 effort=0 velocity=8.7266 -> lower=-0.349 upper=1.5707 effort=0 velocity=0; parent left_middle_link_0 -> left_middle_link0
- joint left_middle_j2: child left_middle_link_2 -> left_middle_link2; limit lower=-0.0873 upper=1.745 effort=0 velocity=8.7266 -> lower=-0.0872 upper=1.7453 effort=0 velocity=0; parent left_middle_link_1 -> left_middle_link1
- joint left_middle_j3: child left_middle_link_3 -> left_middle_link3; limit lower=-0.0873 upper=1.745 effort=0 velocity=8.7266 -> lower=-0.0872 upper=1.7453 effort=0 velocity=0; parent left_middle_link_2 -> left_middle_link2
- joint left_pinky_j0: child left_pinky_link_0 -> left_pinky_link0; limit lower=-0.436 upper=0.436 effort=0 velocity=8.7266 -> lower=-0.4363 upper=0.4363 effort=0 velocity=0; origin xyz=0.0069979 0.034504 0.1125 rpy=3.1416 -1.5708 0 -> xyz=0.0071 0.034504 0.1158 rpy=0 -1.5708 3.1416; parent left_palm_link -> left_palm_base
- joint left_pinky_j1: child left_pinky_link_1 -> left_pinky_link1; limit lower=-0.349 upper=1.5708 effort=0 velocity=8.7266 -> lower=-0.349 upper=1.5707 effort=0 velocity=0; parent left_pinky_link_0 -> left_pinky_link0
- joint left_pinky_j2: child left_pinky_link_2 -> left_pinky_link2; limit lower=-0.0873 upper=1.745 effort=0 velocity=8.7266 -> lower=-0.0872 upper=1.7453 effort=0 velocity=0; origin xyz=0.045 0 0 rpy=0 -4.2275E-05 0 -> xyz=0.045 0 0 rpy=0 0 0; parent left_pinky_link_1 -> left_pinky_link1
- joint left_pinky_j3: child left_pinky_link_3 -> left_pinky_link3; limit lower=-0.0873 upper=1.745 effort=0 velocity=8.7266 -> lower=-0.0872 upper=1.7453 effort=0 velocity=0; parent left_pinky_link_2 -> left_pinky_link2
- joint left_ring_j0: child left_ring_link_0 -> left_ring_link0; limit lower=-0.436 upper=0.436 effort=0 velocity=8.7266 -> lower=-0.4363 upper=0.4363 effort=0 velocity=0; origin xyz=0.0069979 0.011503 0.1155 rpy=3.1416 -1.5708 0 -> xyz=0.0071 0.011503 0.1188 rpy=0 -1.5708 3.14159; parent left_palm_link -> left_palm_base
- joint left_ring_j1: child left_ring_link_1 -> left_ring_link1; limit lower=-0.349 upper=1.5708 effort=0 velocity=8.7266 -> lower=-0.349 upper=1.5707 effort=0 velocity=0; parent left_ring_link_0 -> left_ring_link0
- joint left_ring_j2: child left_ring_link_2 -> left_ring_link2; limit lower=-0.0873 upper=1.745 effort=0 velocity=8.7266 -> lower=-0.0872 upper=1.7453 effort=0 velocity=0; parent left_ring_link_1 -> left_ring_link1
- joint left_ring_j3: child left_ring_link_3 -> left_ring_link3; limit lower=-0.0873 upper=1.745 effort=0 velocity=8.7266 -> lower=-0.0872 upper=1.7453 effort=0 velocity=0; parent left_ring_link_2 -> left_ring_link2
- joint left_thumb_j0: child left_thumb_link_0 -> left_thumb_link0; limit lower=0 upper=1.3963 effort=0 velocity=8.7266 -> lower=0 upper=1.5707 effort=0 velocity=0; origin xyz=0.012998 -0.022996 0.0493 rpy=0 0 -1.5708 -> xyz=0.013 -0.023 0.0493 rpy=0 0 -1.5708; parent left_palm_link -> left_palm_base
- joint left_thumb_j1: child left_thumb_link_1 -> left_thumb_link1; limit lower=-0.1745 upper=1.047 effort=0 velocity=8.7266 -> lower=-0.1745 upper=1.0471 effort=0 velocity=0; parent left_thumb_link_0 -> left_thumb_link0
- joint left_thumb_j2: child left_thumb_link_2 -> left_thumb_link2; limit lower=0 upper=1.396 effort=0 velocity=8.7266 -> lower=0 upper=1.396 effort=0 velocity=0; parent left_thumb_link_1 -> left_thumb_link1
- joint left_thumb_j3: child left_thumb_link_3 -> left_thumb_link3; limit lower=-0.349 upper=1.396 effort=0 velocity=8.7266 -> lower=-0.349 upper=1.396 effort=0 velocity=0; parent left_thumb_link_2 -> left_thumb_link2
- joint left_thumb_j4: child left_thumb_link_4 -> left_thumb_link4; limit lower=-0.349 upper=1.396 effort=0 velocity=8.7266 -> lower=-0.349 upper=1.396 effort=0 velocity=0; parent left_thumb_link_3 -> left_thumb_link3
