Commit message: Updated URDF files for new ApexHand version

File: apex_hand_right/apex_hand_right.urdf (robot description, URDF)
Before this commit: robot right_apex_hand, 47 links, 46 joints
Links:
- removed link right_index_link_0
- removed link right_index_link_1
- removed link right_index_link_2
- removed link right_index_link_3
- removed link right_index_tactile_0
- removed link right_index_tactile_1
- removed link right_index_tactile_2
- removed link right_middle_link_0
- removed link right_middle_link_1
- removed link right_middle_link_2
- removed link right_middle_link_3
- removed link right_middle_tactile_0
- removed link right_middle_tactile_1
- removed link right_middle_tactile_2
- removed link right_pinky_link_0
- removed link right_pinky_link_1
- removed link right_pinky_link_2
- removed link right_pinky_link_3
- removed link right_pinky_tactile_0
- removed link right_pinky_tactile_1
- removed link right_pinky_tactile_2
- removed link right_ring_link_0
- removed link right_ring_link_1
- removed link right_ring_link_2
- removed link right_ring_link_3
- removed link right_ring_tactile_0
- removed link right_ring_tactile_1
- removed link right_ring_tactile_2
- removed link right_thumb_link_0
- removed link right_thumb_link_1
- removed link right_thumb_link_2
- removed link right_thumb_link_3
- removed link right_thumb_link_4
- removed link right_thumb_tactile_0
- removed link right_thumb_tactile_1
- removed link right_thumb_tactile_2
- added link right_index_link0, mass 0.018794; collision mesh filename=./meshes/right_index_link0.STL; visual mesh filename=./meshes/right_index_link0.STL
- added link right_index_link1, mass 0.029095; collision mesh filename=./meshes/right_index_link1.STL; visual mesh filename=./meshes/right_index_link1.STL
- added link right_index_link2, mass 0.011142; collision mesh filename=./meshes/right_index_link2.STL; visual mesh filename=./meshes/right_index_link2.STL
- added link right_index_link3, mass 0.005232; collision mesh filename=./meshes/right_index_link3.STL; visual mesh filename=./meshes/right_index_link3.STL
- added link right_index_tactile0, mass 0.008926; collision mesh filename=./meshes/right_index_tactile0.STL; visual mesh filename=./meshes/right_index_tactile0.STL
- added link right_index_tactile1, mass 0.003635; collision mesh filename=./meshes/right_index_tactile1.STL; visual mesh filename=./meshes/right_index_tactile1.STL
- added link right_index_tactile2, mass 0.009866; collision mesh filename=./meshes/right_index_tactile2.STL; visual mesh filename=./meshes/right_index_tactile2.STL
- added link right_middle_link0, mass 0.018794; collision mesh filename=./meshes/right_middle_link0.STL; visual mesh filename=./meshes/right_middle_link0.STL
- added link right_middle_link1, mass 0.029095; collision mesh filename=./meshes/right_middle_link1.STL; visual mesh filename=./meshes/right_middle_link1.STL
- added link right_middle_link2, mass 0.011142; collision mesh filename=./meshes/right_middle_link2.STL; visual mesh filename=./meshes/right_middle_link2.STL
- added link right_middle_link3, mass 0.005232; collision mesh filename=./meshes/right_middle_link3.STL; visual mesh filename=./meshes/right_middle_link3.STL
- added link right_middle_tactile0, mass 0.008926; collision mesh filename=./meshes/right_middle_tactile0.STL; visual mesh filename=./meshes/right_middle_tactile0.STL
- added link right_middle_tactile1, mass 0.003635; collision mesh filename=./meshes/right_middle_tactile1.STL; visual mesh filename=./meshes/right_middle_tactile1.STL
- added link right_middle_tactile2, mass 0.009866; collision mesh filename=./meshes/right_middle_tactile2.STL; visual mesh filename=./meshes/right_middle_tactile2.STL
- added link right_palm_base, mass 0.1; collision mesh filename=./meshes/right_palm_base.STL; visual mesh filename=./meshes/right_palm_base.STL
- added link right_palm_tactile, mass 0; collision mesh filename=./meshes/right_palm_tactile.STL; visual mesh filename=./meshes/right_palm_tactile.STL
- added link right_pinky_link0, mass 0.018794; collision mesh filename=./meshes/right_pinky_link0.STL; visual mesh filename=./meshes/right_pinky_link0.STL
- added link right_pinky_link1, mass 0.029095; collision mesh filename=./meshes/right_pinky_link1.STL; visual mesh filename=./meshes/right_pinky_link1.STL
- added link right_pinky_link2, mass 0.011142; collision mesh filename=./meshes/right_pinky_link2.STL; visual mesh filename=./meshes/right_pinky_link2.STL
- added link right_pinky_link3, mass 0.005232; collision mesh filename=./meshes/right_pinky_link3.STL; visual mesh filename=./meshes/right_pinky_link3.STL
- added link right_pinky_tactile0, mass 0.008926; collision mesh filename=./meshes/right_pinky_tactile0.STL; visual mesh filename=./meshes/right_pinky_tactile0.STL
- added link right_pinky_tactile1, mass 0.003635; collision mesh filename=./meshes/right_pinky_tactile1.STL; visual mesh filename=./meshes/right_pinky_tactile1.STL
- added link right_pinky_tactile2, mass 0.009866; collision mesh filename=./meshes/right_pinky_tactile2.STL; visual mesh filename=./meshes/right_pinky_tactile2.STL
- added link right_ring_link0, mass 0.018794; collision mesh filename=./meshes/right_ring_link0.STL; visual mesh filename=./meshes/right_ring_link0.STL
- added link right_ring_link1, mass 0.029095; collision mesh filename=./meshes/right_ring_link1.STL; visual mesh filename=./meshes/right_ring_link1.STL
- added link right_ring_link2, mass 0.011142; collision mesh filename=./meshes/right_ring_link2.STL; visual mesh filename=./meshes/right_ring_link2.STL
- added link right_ring_link3, mass 0.005232; collision mesh filename=./meshes/right_ring_link3.STL; visual mesh filename=./meshes/right_ring_link3.STL
- added link right_ring_tactile0, mass 0.008926; collision mesh filename=./meshes/right_ring_tactile0.STL; visual mesh filename=./meshes/right_ring_tactile0.STL
- added link right_ring_tactile1, mass 0.003635; collision mesh filename=./meshes/right_ring_tactile1.STL; visual mesh filename=./meshes/right_ring_tactile1.STL
- added link right_ring_tactile2, mass 0.009866; collision mesh filename=./meshes/right_ring_tactile2.STL; visual mesh filename=./meshes/right_ring_tactile2.STL
- added link right_thumb_link0, mass 0.01096758; collision mesh filename=./meshes/right_thumb_link0.STL; visual mesh filename=./meshes/right_thumb_link0.STL
- added link right_thumb_link1, mass 0.01551203; collision mesh filename=./meshes/right_thumb_link1.STL; visual mesh filename=./meshes/right_thumb_link1.STL
- added link right_thumb_link2, mass 0.0324231; collision mesh filename=./meshes/right_thumb_link2.STL; visual mesh filename=./meshes/right_thumb_link2.STL
- added link right_thumb_link3, mass 0.018383721; collision mesh filename=./meshes/right_thumb_link3.STL; visual mesh filename=./meshes/right_thumb_link3.STL
- added link right_thumb_link4, mass 0.007655847; collision mesh filename=./meshes/right_thumb_link4.STL; visual mesh filename=./meshes/right_thumb_link4.STL
- added link right_thumb_tactile0, mass 0.035995576; collision mesh filename=./meshes/right_thumb_tactile0.STL; visual mesh filename=./meshes/right_thumb_tactile0.STL
- added link right_thumb_tactile1, mass 0.0093845355; collision mesh filename=./meshes/right_thumb_tactile1.STL; visual mesh filename=./meshes/right_thumb_tactile1.STL
- added link right_thumb_tactile2, mass 0.0098665; collision mesh filename=./meshes/right_thumb_tactile2.STL; visual mesh filename=./meshes/right_thumb_tactile2.STL
- link right_index_pad: mass 8.20481262582146E-06 -> 7.85398163397449E-07
- link right_index_tip: mass 8.20481262582146E-06 -> 9.81747704246811E-08
- link right_middle_pad: mass 8.20481262582145E-06 -> 7.85398163397448E-07
- link right_middle_tip: mass 8.20481262582146E-06 -> 9.81747704246811E-08
- link right_palm_link: mass 0.262735816921321 -> 0.2
- link right_pinky_pad: mass 8.20481262582142E-06 -> 7.85398163397449E-07
- link right_pinky_tip: mass 8.20481262582146E-06 -> 9.81747704246811E-08
- link right_ring_pad: mass 8.20481262582145E-06 -> 7.85398163397448E-07
- link right_ring_tip: mass 8.20481262582144E-06 -> 9.81747704246808E-08
- link right_thumb_pad: mass 8.20481262582145E-06 -> 3.927E-07
- link right_thumb_tip: mass 8.20481262582145E-06 -> 4.90873852123406E-08
Joints:
- removed joint right_index_j1_sensor
- removed joint right_index_j2_sensor
- removed joint right_index_j3_sensor
- removed joint right_index_pad
- removed joint right_index_tip
- removed joint right_middle_j1_sensor
- removed joint right_middle_j2_sensor
- removed joint right_middle_j3_sensor
- removed joint right_middle_pad
- removed joint right_middle_tip
- removed joint right_pinky_j1_sensor
- removed joint right_pinky_j3_sensor
- removed joint right_pinky_pad
- removed joint right_pinky_tactile_1
- removed joint right_pinky_tip
- removed joint right_ring_j2_sensor
- removed joint right_ring_j3_sensor
- removed joint right_ring_pad
- removed joint right_ring_tactile_0
- removed joint right_ring_tip
- removed joint right_thumb_j2_sensor
- removed joint right_thumb_j3_sensor
- removed joint right_thumb_j4_sensor
- removed joint right_thumb_pad
- removed joint right_thumb_tip
- added joint right_index_pad_fix: type fixed, parent right_index_tactile2, child right_index_pad, origin xyz=0.017096 0.0071955 0 rpy=0 0 0, axis 0 0 0
- added joint right_index_tactile0_fix: type fixed, parent right_index_link1, child right_index_tactile0, origin xyz=0 0 0 rpy=0 0 0, axis 0 0 0
- added joint right_index_tactile1_fix: type fixed, parent right_index_link2, child right_index_tactile1, origin xyz=0 0 0 rpy=0 0 0, axis 0 0 0
- added joint right_index_tactile2_fix: type fixed, parent right_index_link3, child right_index_tactile2, origin xyz=0 0 0 rpy=0 0 0, axis 0 0 0
- added joint right_index_tip_fix: type fixed, parent right_index_tactile2, child right_index_tip, origin xyz=0.027672 0.00055028 0 rpy=0 0 0, axis 0 0 0
- added joint right_middle_pad_fix: type fixed, parent right_middle_tactile2, child right_middle_pad, origin xyz=0.017096144759137 0.00719554486026074 0 rpy=0 0 0, axis 0 0 0
- added joint right_middle_tactile0_fix: type fixed, parent right_middle_link1, child right_middle_tactile0, origin xyz=0 0 0 rpy=0 0 0, axis 0 0 0
- added joint right_middle_tactile1_fix: type fixed, parent right_middle_link2, child right_middle_tactile1, origin xyz=0 0 0 rpy=0 0 0, axis 0 0 0
- added joint right_middle_tactile2_fix: type fixed, parent right_middle_link3, child right_middle_tactile2, origin xyz=0 0 0 rpy=0 0 0, axis 0 0 0
- added joint right_middle_tip_fix: type fixed, parent right_middle_tactile2, child right_middle_tip, origin xyz=0.027672166719793 0.000550277924150981 0 rpy=0 0 0, axis 0 0 0
- added joint right_palm_base_fix: type fixed, parent right_palm_link, child right_palm_base, origin xyz=0 0 0 rpy=0 0 0, axis 0 0 0
- added joint right_palm_tactile_fix: type fixed, parent right_palm_link, child right_palm_tactile, origin xyz=0 0 0 rpy=0 0 0, axis 0 0 0
- added joint right_pinky_pad_fix: type fixed, parent right_pinky_tactile2, child right_pinky_pad, origin xyz=0.017096 0.0071955 0 rpy=0 0 0, axis 0 0 0
- added joint right_pinky_tactile0_fix: type fixed, parent right_pinky_link1, child right_pinky_tactile0, origin xyz=0 0 0 rpy=0 0 0, axis 0 0 0
- added joint right_pinky_tactile1_fix: type fixed, parent right_pinky_link2, child right_pinky_tactile1, origin xyz=0 0 0 rpy=0 0 0, axis 0 0 0
- added joint right_pinky_tactile2_fix: type fixed, parent right_pinky_link3, child right_pinky_tactile2, origin xyz=0 0 0 rpy=0 0 0, axis 0 0 0
- added joint right_pinky_tip_fix: type fixed, parent right_pinky_tactile2, child right_pinky_tip, origin xyz=0.027672 0.00055028 0 rpy=0 0 0, axis 0 0 0
- added joint right_ring_pad_fix: type fixed, parent right_ring_tactile2, child right_ring_pad, origin xyz=0.017096144759137 0.00719554486026074 0 rpy=0 0 0, axis 0 0 0
- added joint right_ring_tactile0_fix: type fixed, parent right_ring_link1, child right_ring_tactile0, origin xyz=0 0 0 rpy=0 0 0, axis 0 0 0
- added joint right_ring_tactile1_fix: type fixed, parent right_ring_link2, child right_ring_tactile1, origin xyz=0 0 0 rpy=0 0 0, axis 0 0 0
- added joint right_ring_tactile2_fix: type fixed, parent right_ring_link3, child right_ring_tactile2, origin xyz=0 0 0 rpy=0 0 0, axis 0 0 0
- added joint right_ring_tip_fix: type fixed, parent right_ring_tactile2, child right_ring_tip, origin xyz=0.027672166719793 0.000550277924150982 0 rpy=0 0 0, axis 0 0 0
- added joint right_thumb_pad_fix: type fixed, parent right_thumb_tactile2, child right_thumb_pad, origin xyz=0.018471 0.0088124 0 rpy=0 0 0, axis 0 0 0
- added joint right_thumb_tactile0_fix: type fixed, parent right_thumb_link2, child right_thumb_tactile0, origin xyz=0 0 0 rpy=0 0 0, axis 0 0 0
- added joint right_thumb_tactile1_fix: type fixed, parent right_thumb_link3, child right_thumb_tactile1, origin xyz=0 0 0 rpy=0 0 0, axis 0 0 0
- added joint right_thumb_tactile2_fix: type fixed, parent right_thumb_link4, child right_thumb_tactile2, origin xyz=0 0 0 rpy=0 0 0, axis 0 0 0
- added joint right_thumb_tip_fix: type fixed, parent right_thumb_tactile2, child right_thumb_tip, origin xyz=0.029863 -0.00039744 0 rpy=0 0 0, axis 0 0 0
- joint right_index_j0: child right_index_link_0 -> right_index_link0; limit lower=-0.436 upper=0.436 effort=0 velocity=8.7266 -> lower=-0.4363 upper=0.4363 effort=0 velocity=0; origin xyz=0.0069979 0.034496 0.1155 rpy=0 -1.5708 0 -> xyz=0.0071 0.034496 0.1188 rpy=0 -1.5708 0; parent right_palm_link -> right_palm_base
- joint right_index_j1: child right_index_link_1 -> right_index_link1; limit lower=-0.349 upper=1.5708 effort=0 velocity=8.7266 -> lower=-0.349 upper=1.5707 effort=0 velocity=0; origin xyz=0.016 0 0 rpy=-1.570795877559 0 0 -> xyz=0.016 0 0 rpy=-1.5708 0 0; parent right_index_link_0 -> right_index_link0
- joint right_index_j2: child right_index_link_2 -> right_index_link2; limit lower=-0.0873 upper=1.745 effort=0 velocity=8.7266 -> lower=-0.0872 upper=1.7453 effort=0 velocity=0; parent right_index_link_1 -> right_index_link1
- joint right_index_j3: child right_index_link_3 -> right_index_link3; limit lower=-0.0873 upper=1.745 effort=0 velocity=8.7266 -> lower=-0.0872 upper=1.7453 effort=0 velocity=0; parent right_index_link_2 -> right_index_link2
- joint right_middle_j0: child right_middle_link_0 -> right_middle_link0; limit lower=-0.436 upper=0.436 effort=0 velocity=8.7266 -> lower=-0.4363 upper=0.4363 effort=0 velocity=0; origin xyz=0.0069979 0.011496 0.1185 rpy=0 -1.5708 0 -> xyz=0.0071 0.011496 0.1218 rpy=0 -1.5708 0; parent right_palm_link -> right_palm_base
- joint right_middle_j1: child right_middle_link_1 -> right_middle_link1; limit lower=-0.349 upper=1.5708 effort=0 velocity=8.7266 -> lower=-0.349 upper=1.5707 effort=0 velocity=0; parent right_middle_link_0 -> right_middle_link0
- joint right_middle_j2: child right_middle_link_2 -> right_middle_link2; limit lower=-0.0873 upper=1.745 effort=0 velocity=8.7266 -> lower=-0.0872 upper=1.7453 effort=0 velocity=0; origin xyz=0.045 0 0 rpy=0 0 -0.0004769 -> xyz=0.045 0 0 rpy=0 0 0; parent right_middle_link_1 -> right_middle_link1
- joint right_middle_j3: child right_middle_link_3 -> right_middle_link3; limit lower=-0.0873 upper=1.745 effort=0 velocity=8.7266 -> lower=-0.0872 upper=1.7453 effort=0 velocity=0; origin xyz=0.025 1.1923E-05 0 rpy=0 0 0.0004769 -> xyz=0.025 0 0 rpy=0 0 0; parent right_middle_link_2 -> right_middle_link2
- joint right_pinky_j0: child right_pinky_link_0 -> right_pinky_link0; limit lower=-0.436 upper=0.436 effort=0 velocity=8.7266 -> lower=-0.4363 upper=0.4363 effort=0 velocity=0; origin xyz=0.0069979 -0.034504 0.1125 rpy=0 -1.5708 0 -> xyz=0.0071 -0.034504 0.1158 rpy=0 -1.5708 0; parent right_palm_link -> right_palm_base
- joint right_pinky_j1: child right_pinky_link_1 -> right_pinky_link1; limit lower=-0.349 upper=1.5708 effort=0 velocity=8.7266 -> lower=-0.349 upper=1.5707 effort=0 velocity=0; parent right_pinky_link_0 -> right_pinky_link0
- joint right_pinky_j2: child right_pinky_link_2 -> right_pinky_link2; limit lower=-0.0873 upper=1.745 effort=0 velocity=8.7266 -> lower=-0.0872 upper=1.7453 effort=0 velocity=0; origin xyz=0.045 0 0 rpy=0 0 -0.0004769 -> xyz=0.045 0 0 rpy=0 0 0; parent right_pinky_link_1 -> right_pinky_link1
- joint right_pinky_j3: child right_pinky_link_3 -> right_pinky_link3; limit lower=-0.0873 upper=1.745 effort=0 velocity=8.7266 -> lower=-0.0872 upper=1.7453 effort=0 velocity=0; origin xyz=0.025 1.1923E-05 0 rpy=0 0 0 -> xyz=0.025 0 0 rpy=0 0 0; parent right_pinky_link_2 -> right_pinky_link2
- joint right_ring_j0: child right_ring_link_0 -> right_ring_link0; limit lower=-0.436 upper=0.436 effort=0 velocity=8.7266 -> lower=-0.4363 upper=0.4363 effort=0 velocity=0; origin xyz=0.0069979 -0.011503 0.1155 rpy=0 -1.5708 0 -> xyz=0.0071 -0.011503 0.1188 rpy=0 -1.5708 0; parent right_palm_link -> right_palm_base
- joint right_ring_j1: child right_ring_link_1 -> right_ring_link1; limit lower=-0.349 upper=1.5708 effort=0 velocity=8.7266 -> lower=-0.349 upper=1.5707 effort=0 velocity=0; origin xyz=0.016 0 0 rpy=-1.5708 -0.0004769 0 -> xyz=0.016 0 0 rpy=-1.5708 0 0; parent right_ring_link_0 -> right_ring_link0
- joint right_ring_j2: child right_ring_link_2 -> right_ring_link2; limit lower=-0.0873 upper=1.745 effort=0 velocity=8.7266 -> lower=-0.0872 upper=1.7453 effort=0 velocity=0; origin xyz=0.045 2.1461E-05 0 rpy=0 0 0.0004769 -> xyz=0.045 0 0 rpy=0 0 0; parent right_ring_link_1 -> right_ring_link1
- joint right_ring_j3: child right_ring_link_3 -> right_ring_link3; limit lower=-0.0873 upper=1.745 effort=0 velocity=8.7266 -> lower=-0.0872 upper=1.7453 effort=0 velocity=0; parent right_ring_link_2 -> right_ring_link2
- joint right_thumb_j0: child right_thumb_link_0 -> right_thumb_link0; limit lower=0 upper=1.3963 effort=0 velocity=8.7266 -> lower=0 upper=1.5707 effort=0 velocity=0; origin xyz=0.012998 0.022996 0.0493 rpy=3.1416 0 1.5708 -> xyz=0.013 0.023 0.0493 rpy=3.1416 0 1.5708; parent right_palm_link -> right_palm_base
- joint right_thumb_j1: child right_thumb_link_1 -> right_thumb_link1; limit lower=-0.1745 upper=1.047 effort=0 velocity=8.7266 -> lower=-0.1745 upper=1.0471 effort=0 velocity=0; parent right_thumb_link_0 -> right_thumb_link0
- joint right_thumb_j2: child right_thumb_link_2 -> right_thumb_link2; limit lower=0 upper=1.396 effort=0 velocity=8.7266 -> lower=0 upper=1.396 effort=0 velocity=0; parent right_thumb_link_1 -> right_thumb_link1
- joint right_thumb_j3: child right_thumb_link_3 -> right_thumb_link3; limit lower=-0.349 upper=1.396 effort=0 velocity=8.7266 -> lower=-0.349 upper=1.396 effort=0 velocity=0; parent right_thumb_link_2 -> right_thumb_link2
- joint right_thumb_j4: child right_thumb_link_4 -> right_thumb_link4; limit lower=-0.349 upper=1.396 effort=0 velocity=8.7266 -> lower=-0.349 upper=1.396 effort=0 velocity=0; parent right_thumb_link_3 -> right_thumb_link3
